Commit message: feat: Comprehensive GPS-Denied Simulation overhaul with PRM, Informed RRT*, D* Lite, Cascaded PID, Potential Fields, and live FPV telemetry

File: drone_nav_2d/urdf/drone_3d.urdf (robot description, URDF)
Before this commit: robot drone_3d_quadrotor, 10 links, 9 joints
Links:
- added link downward_camera_link, mass 0.05; collision box size=0.04 0.04 0.02; visual box size=0.04 0.04 0.02
Joints:
- added joint downward_camera_joint: type fixed, parent base_link, child downward_camera_link, origin xyz=0 -0.07 0 rpy=-1.5708 0 0
